Commit message: joint continuous mispelled

File: my_robot/urdf/my_robot.xacro (robot description, xacro)
@@ -133,5 +133,5 @@
 		<dynamics damping="1.0" friction="1.0"/>
 	</joint>
-	<joint name="base_to_rwheel" type="continuos">
+	<joint name="base_to_rwheel" type="continuous">
 		<parent link="base_link"/>
 		<child link="rwheel"/>

Commit message: urdf fixed

File: my_robot/urdf/my_robot.xacro (robot description, xacro)
@@ -18,11 +18,54 @@
 	</material>
 	<!-- Links -->
-	<link name="base_link">
-		<visual>
+	<link name="robot_footprint"></link>
+	<link name='base_link'>
+		<pose>0 0 0.1 0 0 0</pose>
+		<inertial>
+			<mass value="15.0"/>
+			<origin xyz="0.0 0 0" rpy=" 0 0 0"/>
+			<inertia
+          ixx="0.1" ixy="0" ixz="0"
+          iyy="0.1" iyz="0"
+          izz="0.1"
+      />
+		</inertial>
+		<collision name='collision'>
+			<origin xyz="0 0 0" rpy=" 0 0 0"/>
 			<geometry>
-				<box size="0.16 0.16 0.12"/>
+				<box size=".4 .2 .1"/>
 			</geometry>
-			<origin rpy="0 0 0" xyz="0 0 0.085"/>
+		</collision>
+		<visual name='chassis_visual'>
+			<origin xyz="0 0 0" rpy=" 0 0 0"/>
+			<geometry>
+				<box size=".4 .2 .1"/>
+			</geometry>
 			<material name="white"/>
+		</visual>
+		<collision name='back_caster_collision'>
+			<origin xyz="-0.15 0 -0.05" rpy=" 0 0 0"/>
+			<geometry>
+				<sphere radius="0.0499"/>
+			</geometry>
+		</collision>
+		<visual name='back_caster_visual'>
+			<origin xyz="-0.15 0 -0.05" rpy=" 0 0 0"/>
+			<geometry>
+				<sphere radius="0.05"/>
+			</geometry>
+			<material name="blue"/>
+		</visual>
+		<collision name='front_caster_collision'>
+			<origin xyz="0.15 0 -0.05" rpy=" 0 0 0"/>
+			<geometry>
+				<sphere radius="0.0499"/>
+			</geometry>
+		</collision>
+		<visual name='front_caster_visual'>
+			<origin xyz="0.15 0 -0.05" rpy=" 0 0 0"/>
+			<geometry>
+				<sphere radius="0.05"/>
+			</geometry>
+			<material name="blue"/>
 		</visual>
 	</link>
@@ -58,22 +101,4 @@
 					izz="0.1" />
 		</inertial>
-	</link>
-	<link name="fwheel_attach">
-		<visual>
-			<geometry>
-				<cylinder length="0.10" radius="0.023"/>
-			</geometry>
-			<origin rpy="0 0 0" xyz="-0.08 0 0"/>
-			<material name="white"/>
-		</visual>
-	</link>
-	<link name="fwheel">
-		<visual>
-			<geometry>
-				<cylinder length="0.005" radius="0.025"/>
-			</geometry>
-			<origin rpy="${PI/2} ${PI/2} 0" xyz="-0.08 0 -0.05"/>
-			<material name="black"/>
-		</visual>
 	</link>
 	<link name="camera_link">
@@ -125,8 +150,13 @@
 	</link>
 	<!-- Joints -->
+	<joint name="robot_footprint_joint" type="fixed">
+		<origin xyz="0 0 0" rpy="0 0 0" />
+		<parent link="robot_footprint"/>
+		<child link="base_link" />
+	</joint>
 	<joint name="base_to_lwheel" type="continuous">
 		<parent link="base_link"/>
 		<child link="lwheel"/>
-		<origin xyz="0 0.115 0.046" rpy="1.5708 0 0"/>
+		<origin xyz="0 0.15 0" rpy="0 0 0"/>
 		<axis xyz="0 1 0" rpy="0 0 0"/>
 		<limit effort="10000" velocity="1000"/>
@@ -136,22 +166,12 @@
 		<parent link="base_link"/>
 		<child link="rwheel"/>
-		<origin xyz="0 -0.115 0.046" rpy="-1.5708 0 0"/>
+		<origin xyz="0 -0.15 0" rpy="-{PI/2} 0 0"/>
 		<axis xyz="0 1 0" rpy="0 0 0"/>
 		<limit effort="10000" velocity="1000"/>
 		<dynamics damping="1.0" friction="1.0"/>
 	</joint>
-	<joint name="base_to_fattach" type="fixed">
-		<parent link="base_link"/>
-		<child link="fwheel_attach"/>
-		<origin xyz="0 0 0" rpy="0 0 0"/>
-	</joint>
-	<joint name="fattach_to_fwheel" type="fixed">
-		<parent link="fwheel_attach"/>
-		<child link="fwheel"/>
-		<origin xyz="0 0 0" rpy="0 0 0"/>
-	</joint>
 	<joint name="camera_joint" type="fixed">
 		<axis xyz="0 1 0" />
-		<origin xyz="0.2 0 0" rpy="0 -${PI/2} 0"/>
+		<origin xyz="0.2 0 0" rpy="0 0 0"/>
 		<parent link="base_link"/>
 		<child link="camera_link"/>

Commit message: fixed wheels urdf

File: my_robot/urdf/my_robot.xacro (robot description, xacro)
@@ -78,4 +78,10 @@
 			<material name="black"/>
 		</visual>
+		<collision>
+			<geometry>
+				<cylinder length="0.05" radius="0.15"/>
+			</geometry>
+			<origin rpy="0 0 0" xyz="0 0 0"/>
+		</collision>
 		<inertial>
 			<mass value="5" />
@@ -94,4 +100,10 @@
 			<material name="black"/>
 		</visual>
+		<collision>
+			<geometry>
+				<cylinder length="0.05" radius="0.15"/>
+			</geometry>
+			<origin rpy="0 0 0" xyz="0 0 0"/>
+		</collision>
 		<inertial>
 			<mass value="5" />
@@ -106,5 +118,4 @@
 			<origin xyz="0 0 0" rpy="0 0 0"/>
 			<geometry>
-				<!--mesh filename="package://simple_arm/meshes/camera.dae"/-->
 				<sphere radius="0.005"/>
 			</geometry>
@@ -130,5 +141,4 @@
 			<origin xyz="0 0 0" rpy="0 0 0"/>
 			<geometry>
-				<mesh filename = "package://my_robot/meshes/hokuyo.dae"/>
 				<box size="0.1 0.1 0.1"/>
 			</geometry>
@@ -158,5 +168,5 @@
 		<parent link="base_link"/>
 		<child link="lwheel"/>
-		<origin xyz="0 0.15 0" rpy="0 0 0"/>
+		<origin xyz="0 0.15 0" rpy="-${PI/2} 0 0"/>
 		<axis xyz="0 1 0" rpy="0 0 0"/>
 		<limit effort="10000" velocity="1000"/>
@@ -166,5 +176,5 @@
 		<parent link="base_link"/>
 		<child link="rwheel"/>
-		<origin xyz="0 -0.15 0" rpy="-{PI/2} 0 0"/>
+		<origin xyz="0 -0.15 0" rpy="-${PI/2} 0 0"/>
 		<axis xyz="0 1 0" rpy="0 0 0"/>
 		<limit effort="10000" velocity="1000"/>

Commit message: fix: corrected urdf dimension and plugin

File: my_robot/urdf/my_robot.xacro (robot description, xacro)
@@ -73,5 +73,5 @@
 		<visual>
 			<geometry>
-				<cylinder length="0.05" radius="0.15"/>
+				<cylinder length="0.05" radius="0.1"/>
 			</geometry>
 			<origin rpy="0 0 0" xyz="0 0 0"/>
@@ -80,5 +80,5 @@
 		<collision>
 			<geometry>
-				<cylinder length="0.05" radius="0.15"/>
+				<cylinder length="0.05" radius="0.1"/>
 			</geometry>
 			<origin rpy="0 0 0" xyz="0 0 0"/>
@@ -95,5 +95,5 @@
 		<visual>
 			<geometry>
-				<cylinder length="0.05" radius="0.15"/>
+				<cylinder length="0.05" radius="0.1"/>
 			</geometry>
 			<origin rpy="0 0 0" xyz="0 0 0"/>
@@ -102,5 +102,5 @@
 		<collision>
 			<geometry>
-				<cylinder length="0.05" radius="0.15"/>
+				<cylinder length="0.05" radius="0.1"/>
 			</geometry>
 			<origin rpy="0 0 0" xyz="0 0 0"/>
@@ -118,5 +118,5 @@
 			<origin xyz="0 0 0" rpy="0 0 0"/>
 			<geometry>
-				<sphere radius="0.005"/>
+				<box size="0.05 0.05 0.05"/>
 			</geometry>
 		</collision>
@@ -125,5 +125,5 @@
 			<geometry>
 				<!--mesh filename="package://my_robot/meshes/camera.dae"/-->
-				<sphere radius="0.05"/>
+				<box size="0.05 0.05 0.05"/>
 			</geometry>
 			<material name="red"/>
@@ -169,5 +169,5 @@
 		<child link="lwheel"/>
 		<origin xyz="0 0.15 0" rpy="-${PI/2} 0 0"/>
-		<axis xyz="0 1 0" rpy="0 0 0"/>
+		<axis xyz="0 0 1" rpy="0 0 0"/>
 		<limit effort="10000" velocity="1000"/>
 		<dynamics damping="1.0" friction="1.0"/>
@@ -177,5 +177,5 @@
 		<child link="rwheel"/>
 		<origin xyz="0 -0.15 0" rpy="-${PI/2} 0 0"/>
-		<axis xyz="0 1 0" rpy="0 0 0"/>
+		<axis xyz="0 0 1" rpy="0 0 0"/>
 		<limit effort="10000" velocity="1000"/>
 		<dynamics damping="1.0" friction="1.0"/>

Commit message: fix: change name so that plugin and urdf link match

File: my_robot/urdf/my_robot.xacro (robot description, xacro)
@@ -114,5 +114,5 @@
 		</inertial>
 	</link>
-	<link name="camera_link">
+	<link name="camera">
 		<collision>
 			<origin xyz="0 0 0" rpy="0 0 0"/>
@@ -137,5 +137,5 @@
 		</inertial>
 	</link>
-	<link name="hokuyo_link">
+	<link name="hokuyo">
 		<collision>
 			<origin xyz="0 0 0" rpy="0 0 0"/>
@@ -185,9 +185,9 @@
 		<origin xyz="0.2 0 0" rpy="0 0 0"/>
 		<parent link="base_link"/>
-		<child link="camera_link"/>
+		<child link="camera"/>
 	</joint>
 	<joint name="hokuyo_joint" type="fixed">
 		<parent link="base_link"/>
-		<child link="hokuyo_link"/>
+		<child link="hokuyo"/>
 		<origin xyz="0.15 0 0.1" rpy="0 0 0"/>
 		<axis xyz="0 1 0" />
